Commit message: completed till building 4 diff cross section without bottom mat

File: sa2_description/urdf/end_effactor.urdf.xacro (robot description, xacro)
@@ -275,3 +275,111 @@
   </joint>
 </xacro:macro>
+<!-- ========================================================= -->
+  <!-- SA3 GRIPPER: SA3_GRPR01.STL                                -->
+  <!-- Mesh: sa2_description/meshes/ee/SA3_GRPR01.STL              -->
+  <!-- ========================================================= -->
+  <xacro:macro name="sa3_grpr01"
+    params="
+      parent_link
+      prefix:=''
+      xyz:='0 0 0'
+      rpy:='0 1.5708 0'
+      visual_xyz:='0 0 0'
+      visual_rpy:='0 -1.5708 0'
+      mesh_scale:='0.001 0.001 0.001'">
+    <link name="${prefix}sa3_grpr01">
+      <!-- Provisional inertial parameters.
+           Replace with measured/CAD-derived values for accurate dynamics. -->
+      <inertial>
+        <origin xyz="0 0 0" rpy="0 0 0"/>
+        <mass value="0.45"/>
+        <inertia
+          ixx="0.00092934"
+          ixy="0.00000034"
+          ixz="-0.00000738"
+          iyy="0.00071447"
+          iyz="0.00000005"
+          izz="0.00039442"/>
+      </inertial>
+      <!-- Visual geometry -->
+      <visual>
+        <origin xyz="${visual_xyz}" rpy="${visual_rpy}"/>
+        <geometry>
+          <mesh
+            filename="package://sa2_description/meshes/ee/SA3_GRPR01.STL"/>
+        </geometry>
+        <material name="${prefix}sa3_grpr01_material">
+          <color rgba="0.792156862745098 0.819607843137255 0.933333333333333 1"/>
+        </material>
+      </visual>
+      <!-- Collision geometry -->
+      <collision>
+        <origin xyz="${visual_xyz}" rpy="${visual_rpy}"/>
+        <geometry>
+          <mesh
+            filename="package://sa2_description/meshes/ee/SA3_GRPR01.STL"/>
+        </geometry>
+      </collision>
+    </link>
+    <!-- Fixed mount to the selected robot link -->
+    <joint name="${prefix}sa3_grpr01_mount" type="fixed">
+      <origin xyz="${xyz}" rpy="${rpy}"/>
+      <parent link="${parent_link}"/>
+      <child link="${prefix}sa3_grpr01"/>
+    </joint>
+  </xacro:macro>
+  <!-- ========================================================= -->
+  <!-- SA3 GRIPPER R: SA3_GRPR01_r.STL                           -->
+  <!-- Intended for Robot 4 only                                 -->
+  <!-- ========================================================= -->
+  <xacro:macro name="sa3_grpr01_r"
+    params="
+      parent_link
+      prefix:=''
+      xyz:='0 0 0'
+      rpy:='0 1.5708 0'
+      visual_xyz:='0 0 0'
+      visual_rpy:='0 -1.5708 0'
+      mesh_scale:='0.001 0.001 0.001'">
+    <link name="${prefix}sa3_grpr01_r">
+      <inertial>
+        <origin xyz="0 0 0" rpy="0 0 0"/>
+        <mass value="0.45"/>
+        <inertia
+          ixx="0.00092934"
+          ixy="0.00000034"
+          ixz="-0.00000738"
+          iyy="0.00071447"
+          iyz="0.00000005"
+          izz="0.00039442"/>
+      </inertial>
+      <!-- Visual geometry -->
+      <visual>
+        <origin xyz="${visual_xyz}" rpy="${visual_rpy}"/>
+        <geometry>
+          <mesh
+            filename="package://sa2_description/meshes/ee/SA3_GRPR01_r.stl"
+            scale="${mesh_scale}"/>
+        </geometry>
+        <material name="${prefix}sa3_grpr01_r_material">
+          <color rgba="0.792156862745098 0.819607843137255 0.933333333333333 1"/>
+        </material>
+      </visual>
+      <!-- Collision geometry -->
+      <collision>
+        <origin xyz="${visual_xyz}" rpy="${visual_rpy}"/>
+        <geometry>
+          <mesh
+            filename="package://sa2_description/meshes/ee/SA3_GRPR01_r.stl"
+            scale="${mesh_scale}"/>
+        </geometry>
+      </collision>
+    </link>
+    <!-- Fixed mount to the selected robot link -->
+    <joint name="${prefix}sa3_grpr01_r_mount" type="fixed">
+      <origin xyz="${xyz}" rpy="${rpy}"/>
+      <parent link="${parent_link}"/>
+      <child link="${prefix}sa3_grpr01_r"/>
+    </joint>
+  </xacro:macro>
 </robot>

File: sa2_description/urdf/robot.urdf.xacro (robot description, xacro)
@@ -11,4 +11,8 @@
   <xacro:arg name="robot4_pedestal_xyz" default="5.6 0.15 0.0"/>
   <xacro:arg name="robot4_pedestal_rpy" default="0 0 -1.5708"/>
+  <!-- Gantry position and orientation: overridden from workcell.yaml -->
+  <xacro:arg name="gantry_xyz" default="0.0 0.0 0.0"/>
+  <xacro:arg name="gantry_rpy" default="0.0 0.0 0.0"/>
+  <xacro:arg name="gantry_scale" default="0.001 0.001 0.001"/>
   <!-- ========================================================= -->
   <!-- ARGUMENTS                                                 -->
@@ -30,4 +34,7 @@
   <xacro:include
     filename="$(find sa2_description)/urdf/end_effactor.urdf.xacro"/>
+  <!-- Gantry -->
+  <xacro:include
+    filename="$(find sa2_description)/urdf/gantry.urdf.xacro"/>
   <!-- ros2_control -->
   <xacro:include
@@ -37,4 +44,9 @@
   <!-- ========================================================= -->
   <link name="world"/>
+  <xacro:sa3_gantry
+    parent="world"
+    xyz="$(arg gantry_xyz)"
+    rpy="$(arg gantry_rpy)"
+    scale="$(arg gantry_scale)"/>
   <!-- ========================================================= -->
   <!-- MATERIALS                                                 -->
@@ -244,5 +256,5 @@
   </xacro:r2000ic_210r>
   <!-- Robot 3 Schunk gripper -->
-  <xacro:schunk_gripper
+  <xacro:sa3_grpr01
     parent_link="robot3_gripper_mount"
     prefix="robot3_"
@@ -260,5 +272,5 @@
   </link>
   <joint name="robot3_end_effactor_joint" type="fixed">
-    <origin xyz="0.2 0 0" rpy="0 0 0"/>
+    <origin xyz="0.3 0 0" rpy="0 0 0"/>
     <parent link="robot3_flange"/>
     <child link="robot3_end_effactor"/>
@@ -301,10 +313,10 @@
     <origin xyz="0.4 0.4 2.1" rpy="0 0 -1.5708"/>
   </xacro:r2000ic_210r>
-  <!-- Robot 4 Schunk gripper -->
-  <xacro:schunk_gripper
+  <!-- Robot 4: SA3_GRPR01_R gripper -->
+  <xacro:sa3_grpr01_r
     parent_link="robot4_gripper_mount"
     prefix="robot4_"
     xyz="0 0 0"
-    rpy="0 1.57 0"/>
+    rpy="0 0 0"/>
   <!-- Robot 4 end effactor (ball, +0.2 m in X from flange) -->
   <link name="robot4_end_effactor">
@@ -318,5 +330,5 @@
   </link>
   <joint name="robot4_end_effactor_joint" type="fixed">
-    <origin xyz="0.2 0 0" rpy="0 0 0"/>
+    <origin xyz="0.3 0 0" rpy="0 0 0"/>
     <parent link="robot4_flange"/>
     <child link="robot4_end_effactor"/>

File: sa2_description/urdf/ros2_controller.urdf.xacro (robot description, xacro)
@@ -79,4 +79,30 @@
     <xacro:controlled_joint name="robot4_J5"/>
     <xacro:controlled_joint name="robot4_J6"/>
+    <!-- ======================================================= -->
+    <!-- GANTRY : HORIZONTAL SLIDE                               -->
+    <!-- ======================================================= -->
+    <joint name="gantry_slide_joint">
+      <command_interface name="position">
+        <param name="min">0.0</param>
+        <param name="max">4.0</param>
+      </command_interface>
+      <state_interface name="position">
+        <param name="initial_value">0.0</param>
+      </state_interface>
+      <state_interface name="velocity"/>
+    </joint>
+    <!-- ======================================================= -->
+    <!-- GANTRY : VERTICAL DOWN MOVEMENT                         -->
+    <!-- ======================================================= -->
+    <joint name="gantry_down_joint">
+      <command_interface name="position">
+        <param name="min">0.0</param>
+        <param name="max">2.0</param>
+      </command_interface>
+      <state_interface name="position">
+        <param name="initial_value">0.0</param>
+      </state_interface>
+      <state_interface name="velocity"/>
+    </joint>
   </ros2_control>
   <!-- ========================================================= -->
