Commit message: 1)added motion sequence yaml for different cross sections. 2)Whole Sub-assembly pick plce working

File: sa2_description/urdf/gantry.urdf.xacro (robot description, xacro)
@@ -1,11 +1,5 @@
 <?xml version="1.0"?>
 <robot xmlns:xacro="http://www.ros.org/wiki/xacro"
-       name="sa3_gantry">
-  <!-- ========================================================= -->
-  <!-- GANTRY PARAMETERS                                         -->
-  <!-- ========================================================= -->
-  <xacro:arg name="gantry_xyz" default="1.3, 0.0, 0.0"/>
-  <xacro:arg name="gantry_rpy" default="0.0 0.0 0.0"/>
-  <xacro:arg name="gantry_scale" default="0.001 0.001 0.001"/>
+       name="sa3_gantry_macro">
   <!-- ========================================================= -->
   <!-- MATERIALS                                                 -->
@@ -13,7 +7,4 @@
   <material name="gantry_rail_material">
     <color rgba="0.25 0.28 0.32 1.0"/>
-  </material>
-  <material name="gantry_carriage_material">
-    <color rgba="0.85 0.45 0.10 1.0"/>
   </material>
   <material name="gantry_part_material">
@@ -28,5 +19,4 @@
     <!-- ======================================================= -->
     <!-- GANTRY FRAME / RAIL                                     -->
-    <!-- Mesh geometry starts at its original STL coordinates.  -->
     <!-- ======================================================= -->
     <link name="gantry_link">
@@ -57,5 +47,5 @@
       </inertial>
     </link>
-    <!-- World placement is controlled by workcell.yaml -->
+    <!-- World placement -->
     <joint name="world_to_gantry" type="fixed">
       <parent link="${parent}"/>
@@ -65,19 +55,7 @@
     <!-- ======================================================= -->
     <!-- HORIZONTAL SLIDING CARRIAGE                             -->
+    <!-- Orange box visual and collision removed                 -->
     <!-- ======================================================= -->
     <link name="gantry_carriage_link">
-      <visual>
-        <origin xyz="0 0 0" rpy="0 0 0"/>
-        <geometry>
-          <box size="0.35 0.35 0.20"/>
-        </geometry>
-        <material name="gantry_carriage_material"/>
-      </visual>
-      <collision>
-        <origin xyz="0 0 0" rpy="0 0 0"/>
-        <geometry>
-          <box size="0.35 0.35 0.20"/>
-        </geometry>
-      </collision>
       <inertial>
         <origin xyz="0 0 0" rpy="0 0 0"/>
@@ -95,6 +73,6 @@
       <axis xyz="1 0 0"/>
       <limit
-          lower="0.0"
-          upper="4.0"
+          lower="-10.6"
+          upper="10.6"
           effort="1000.0"
           velocity="0.5"/>
@@ -103,8 +81,9 @@
     <!-- ======================================================= -->
     <!-- VERTICAL GANTRY PART                                    -->
+    <!-- Mesh visual and collision retained                     -->
     <!-- ======================================================= -->
     <link name="gantry_part_link">
       <visual>
-        <origin xyz="0 0.5 5" rpy="0 0 0"/>
+        <origin xyz="10 0.5 5" rpy="0 0 0"/>
         <geometry>
           <mesh
@@ -115,5 +94,5 @@
       </visual>
       <collision>
-        <origin xyz="0 0.5 5" rpy="0 0 0"/>
+        <origin xyz="10 0.5 5" rpy="0 0 0"/>
         <geometry>
           <mesh
@@ -135,11 +114,11 @@
       <child link="gantry_part_link"/>
       <origin xyz="0 0 0" rpy="0 0 0"/>
-      <!-- Positive motion moves the part downward -->
+      <!-- Positive joint motion moves the part downward -->
       <axis xyz="0 0 -1"/>
       <limit
           lower="0.0"
-          upper="2.0"
+          upper="6.6"
           effort="1000.0"
-          velocity="0.25"/>
+          velocity="0.5"/>
       <dynamics damping="5.0" friction="1.0"/>
     </joint>

File: sa2_description/urdf/robot.urdf.xacro (robot description, xacro)
@@ -11,11 +11,11 @@
   <xacro:arg name="robot4_pedestal_xyz" default="5.6 0.15 0.0"/>
   <xacro:arg name="robot4_pedestal_rpy" default="0 0 -1.5708"/>
+    <!-- ========================================================= -->
+  <!-- ARGUMENTS                                                 -->
+  <!-- ========================================================= -->
   <!-- Gantry position and orientation: overridden from workcell.yaml -->
   <xacro:arg name="gantry_xyz" default="0.0 0.0 0.0"/>
   <xacro:arg name="gantry_rpy" default="0.0 0.0 0.0"/>
   <xacro:arg name="gantry_scale" default="0.001 0.001 0.001"/>
-  <!-- ========================================================= -->
-  <!-- ARGUMENTS                                                 -->
-  <!-- ========================================================= -->
   <xacro:arg name="hardware_mode" default="mock"/>
   <xacro:property
@@ -34,10 +34,9 @@
   <xacro:include
     filename="$(find sa2_description)/urdf/end_effactor.urdf.xacro"/>
-  <!-- Gantry -->
+  <!-- ros2_control -->
+  <xacro:include
+    filename="$(find sa2_description)/urdf/ros2_controller.urdf.xacro"/>
   <xacro:include
     filename="$(find sa2_description)/urdf/gantry.urdf.xacro"/>
-  <!-- ros2_control -->
-  <xacro:include
-    filename="$(find sa2_description)/urdf/ros2_controller.urdf.xacro"/>
   <!-- ========================================================= -->
   <!-- WORLD                                                     -->
@@ -272,7 +271,22 @@
   </link>
   <joint name="robot3_end_effactor_joint" type="fixed">
-    <origin xyz="0.3 0 0" rpy="0 0 0"/>
+    <origin xyz="0.2 0 0" rpy="0 0 0"/>
     <parent link="robot3_flange"/>
     <child link="robot3_end_effactor"/>
+  </joint>
+    <!-- Robot 3 end effactor (ball, +0.2 m in X from flange) -->
+  <link name="robot3_end_effactor_ff">
+    <visual>
+      <origin xyz="0 0 0" rpy="0 0 0"/>
+      <geometry>
+        <sphere radius="0.02"/>
+      </geometry>
+      <material name="end_effactor_material"/>
+    </visual>
+  </link>
+  <joint name="robot3_end_effactor_ff_joint" type="fixed">
+    <origin xyz="0.32 0 0" rpy="0 0 0"/>
+    <parent link="robot3_flange"/>
+    <child link="robot3_end_effactor_ff"/>
   </joint>
   <!-- ========================================================= -->
@@ -314,9 +328,9 @@
   </xacro:r2000ic_210r>
   <!-- Robot 4: SA3_GRPR01_R gripper -->
-  <xacro:sa3_grpr01_r
-    parent_link="robot4_gripper_mount"
-    prefix="robot4_"
-    xyz="0 0 0"
-    rpy="0 0 0"/>
+<xacro:sa3_grpr01_r
+  parent_link="robot4_gripper_mount"
+  prefix="robot4_"
+  xyz="0 0 0"
+  rpy="0 0 0"/>
   <!-- Robot 4 end effactor (ball, +0.2 m in X from flange) -->
   <link name="robot4_end_effactor">
@@ -330,7 +344,21 @@
   </link>
   <joint name="robot4_end_effactor_joint" type="fixed">
-    <origin xyz="0.3 0 0" rpy="0 0 0"/>
+    <origin xyz="0.2 0 0" rpy="0 0 0"/>
     <parent link="robot4_flange"/>
     <child link="robot4_end_effactor"/>
   </joint>
+  <link name="robot4_end_effactor_ff">
+    <visual>
+      <origin xyz="0 0 0" rpy="0 0 0"/>
+      <geometry>
+        <sphere radius="0.02"/>
+      </geometry>
+      <material name="end_effactor_material"/>
+    </visual>
+  </link>
+  <joint name="robot4_end_effactor_ff_joint" type="fixed">
+    <origin xyz="0.32 0 0" rpy="0 0 0"/>
+    <parent link="robot4_flange"/>
+    <child link="robot4_end_effactor_ff"/>
+  </joint>
 </robot>
